File: Wooden_Mirror.kicad_pcb (KiCad board)
At the start: 2 copper layers, 73.7 x 55.9 mm, 25 parts, among them J1 Conn_02x10_Odd_Even, J2 Servo, J3 Programmer, J4 LED_CHAIN, J5 Conn_02x10_Odd_Even, U1 TLV1117-33, U2 MSP430G2233IN20

Commit message: Sent V2
Parts:
- moved R3 37.0 mm to (88.9, 105.4), turned to 90 degrees
- moved U2 34.1 mm to (96.5, 123.4), turned to 90 degrees
- moved R1 31.4 mm to (127.0, 97.8), turned to -90 degrees
- moved C2 30.9 mm to (125.7, 124.5)
- moved J4 29.2 mm to (109.2, 109.2), turned to -90 degrees
- moved JP1 26.0 mm to (95.9, 101.6)
- moved C8 23.8 mm to (107.9, 96.4)
- moved D2 23.8 mm to (108.0, 101.6)
- moved D1 21.3 mm to (120.7, 101.6), turned to 180 degrees
- moved R2 20.6 mm to (127.0, 111.8)
- moved J3 15.8 mm to (88.9, 113.8)
Connections:
- J1 pad 17: unconnected-(J1-Pin_17-Pad17) -> Net-(J1-Pin_17)
- J1 pad 19: unconnected-(J1-Pin_19-Pad19) -> Net-(J1-Pin_19)
- J5 pad 17: unconnected-(J5-Pin_17-Pad17) -> Net-(J5-Pin_17)
- J5 pad 19: unconnected-(J5-Pin_19-Pad19) -> Net-(J5-Pin_19)
- U2 pad 12: unconnected-(U2-P2.4/TA1.2-Pad12) -> Net-(J1-Pin_17)
- U2 pad 13: unconnected-(U2-P2.5/TA1.2-Pad13) -> Net-(J1-Pin_19)
- U2 pad 6: unconnected-(U2-TCK/SMCLK/UCB0STE/UCA0CLK/VREF+/VeREF+/A4/P1.4-Pad6) -> Net-(J5-Pin_17)
- U2 pad 7: unconnected-(U2-TMS/TA0.0/UCB0CLK/UCA0STE/A5/P1.5-Pad7) -> Net-(J5-Pin_19)
Routing:
- net Net-(J1-Pin_17): track 0.00 -> 62.2 mm, vias 0 -> 1
- net Net-(J1-Pin_19): track 0.00 -> 44.3 mm, vias 0 -> 6
- net Net-(J5-Pin_17): track 0.00 -> 34.6 mm
- net Net-(J5-Pin_19): track 0.00 -> 31.0 mm
- net /LED_DOUT: track 66.3 -> 37.1 mm, vias 0 -> 1
- net Net-(U2-P2.0/TA1.0): track 13.8 -> 26.9 mm
- net /SBWTDIO: track 39.9 -> 52.6 mm, vias 6 -> 4
- net Net-(U2-TDO/TDI/UCB0SIMO/UCB0SDA/A7/P1.7): track 16.6 -> 24.6 mm, vias 0 -> 2
- net Net-(J2-Pin_3): track 32.6 -> 39.0 mm, vias 2 -> 3
- net +3V3: track 122.3 -> 117.0 mm, vias 0 -> 2
- net /LED_DIN: track 49.4 -> 45.2 mm, vias 0 -> 3
- net /Serial_OUT: track 57.5 -> 61.1 mm, vias 4 -> 0
- net +5V: track 66.9 -> 63.5 mm
- net /SBWTCK: track 21.3 -> 18.4 mm
- net Net-(JP1-B): track 7.38 -> 9.92 mm
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Other:
- board text added: "EGS 1006 Fall 2024 Wooden Wall v 2.0"

Commit message: V3 sent to JCLPCB
Connections:
- J3 pad 1: +3V3 -> GND
Routing:
- net +3V3: track 117.0 -> 111.7 mm
Other:
- board text added: "+"
- board text added: "+5V"
- board text added: "B"
- board text added: "EGS 1006 Fall 2024 Wooden Wall v 3.0"
- board text added: "GND"
- board text added: "O"
- board text added: "Y"
- board text removed: "EGS 1006 Fall 2024 Wooden Wall v 2.0"
