File: Wooden_Mirror.kicad_sch (KiCad schematic)
At the start: 25 parts, among them J1 Conn_02x10_Odd_Even, J2 Servo, J3 Programmer, J4 LED_CHAIN, J5 Conn_02x10_Odd_Even, U1 TLV1117-33, U2 MSP430G2233IN20

Commit message: Sent V2
Connections:
- net at U2.12 (P2.4/TA1.2): now also J1.17 (Pin_17)
- net at U2.13 (P2.5/TA1.2): now also J1.19 (Pin_19)
- net at U2.6 (TCK/SMCLK/UCB0STE/UCA0CLK/VREF+/VeREF+/A4/P1.4): now also J5.17 (Pin_17)
- net at U2.7 (TMS/TA0.0/UCB0CLK/UCA0STE/A5/P1.5): now also J5.19 (Pin_19)
- no-connect marks 15 -> 7
Changed lines of the file:
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@@
 	)
 	(no_connect
-		(at 40.64 99.06)
-	)
-	(no_connect
-		(at 246.38 101.6)
-	)
-	(no_connect
 		(at 106.68 100.33)
 	)
 	(no_connect
-		(at 40.64 96.52)
-	)
-	(no_connect
-		(at 182.88 90.17)
-	)
-	(no_connect
-		(at 246.38 99.06)
-	)
-	(no_connect
 		(at 106.68 85.09)
 	)
 	(no_connect
-		(at 106.68 92.71)
-	)
-	(no_connect
 		(at 106.68 90.17)
 	)
@@
 		(at 106.68 87.63)
 	)
-	(no_connect
-		(at 182.88 92.71)
-	)
-	(no_connect
-		(at 106.68 95.25)
+	(wire
+		(pts
+			(xy 101.6 95.25) (xy 106.68 95.25)
+		)
+		(stroke
+			(width 0)
+			(type default)
+		)
 	)
 	(wire
@@
 	(wire
 		(pts
+			(xy 40.64 96.52) (xy 36.83 96.52)
+		)
+		(stroke
+			(width 0)
+			(type default)
+		)
+	)
+	(wire
+		(pts
+			(xy 36.83 106.68) (xy 100.33 106.68)
+		)
+		(stroke
+			(width 0)
+			(type default)
+		)
+	)
+	(wire
+		(pts
 			(xy 83.82 44.45) (xy 83.82 45.72)
 		)
@@
 	(wire
 		(pts
+			(xy 100.33 106.68) (xy 100.33 92.71)
+		)
+		(stroke
+			(width 0)
+			(type default)
+		)
+	)
+	(wire
+		(pts
 			(xy 34.29 86.36) (xy 38.1 86.36)
 		)
@@
 	(wire
 		(pts
+			(xy 238.76 101.6) (xy 246.38 101.6)
+		)
+		(stroke
+			(width 0)
+			(type default)
+		)
+	)
+	(wire
+		(pts
 			(xy 259.08 86.36) (xy 261.62 86.36)
 		)
@@
 	(wire
 		(pts
+			(xy 101.6 105.41) (xy 101.6 95.25)
+		)
+		(stroke
+			(width 0)
+			(type default)
+		)
+	)
+	(wire
+		(pts
 			(xy 182.88 82.55) (xy 198.12 82.55)
 		)
@@
 	(wire
 		(pts
+			(xy 36.83 96.52) (xy 36.83 106.68)
+		)
+		(stroke
+			(width 0)
+			(type default)
+		)
+	)
+	(wire
+		(pts
 			(xy 114.3 35.56) (xy 143.51 35.56)
 		)
@@
 	(wire
 		(pts
+			(xy 38.1 99.06) (xy 38.1 105.41)
+		)
+		(stroke
+			(width 0)
+			(type default)
+		)
+	)
+	(wire
+		(pts
 			(xy 243.84 96.52) (xy 243.84 93.98)
 		)
@@
 	(wire
 		(pts
+			(xy 38.1 105.41) (xy 101.6 105.41)
+		)
+		(stroke
+			(width 0)
+			(type default)
+		)
+	)
+	(wire
+		(pts
 			(xy 187.96 97.79) (xy 187.96 124.46)
 		)
@@
 	(wire
 		(pts
+			(xy 182.88 90.17) (xy 241.3 90.17)
+		)
+		(stroke
+			(width 0)
+			(type default)
+		)
+	)
+	(wire
+		(pts
 			(xy 259.08 81.28) (xy 261.62 81.28)
 		)
@@
 	(wire
 		(pts
+			(xy 238.76 92.71) (xy 238.76 101.6)
+		)
+		(stroke
+			(width 0)
+			(type default)
+		)
+	)
+	(wire
+		(pts
 			(xy 146.05 109.22) (xy 146.05 111.76)
 		)
@@
 	(wire
 		(pts
+			(xy 241.3 99.06) (xy 246.38 99.06)
+		)
+		(stroke
+			(width 0)
+			(type default)
+		)
+	)
+	(wire
+		(pts
 			(xy 68.58 34.29) (xy 68.58 35.56)
 		)
@@
 	(wire
 		(pts
+			(xy 100.33 92.71) (xy 106.68 92.71)
+		)
+		(stroke
+			(width 0)
+			(type default)
+		)
+	)
+	(wire
+		(pts
 			(xy 30.48 35.56) (xy 45.72 35.56)
 		)
@@
 	(wire
 		(pts
+			(xy 241.3 90.17) (xy 241.3 99.06)
+		)
+		(stroke
+			(width 0)
+			(type default)
+		)
+	)
+	(wire
+		(pts
 			(xy 55.88 76.2) (xy 58.42 76.2)
 		)
@@
 	(wire
 		(pts
+			(xy 182.88 92.71) (xy 238.76 92.71)
+		)
+		(stroke
+			(width 0)
+			(type default)
+		)
+	)
+	(wire
+		(pts
 			(xy 58.42 35.56) (xy 68.58 35.56)
 		)
@@
 	(wire
 		(pts
+			(xy 40.64 99.06) (xy 38.1 99.06)
+		)
+		(stroke
+			(width 0)
+			(type default)
+		)
+	)
+	(wire
+		(pts
 			(xy 99.06 158.75) (xy 83.82 158.75)
 		)
@@
 	(text_box "P1.7 is used to drive the WS2812B LED module.  The module uses ns timing that needs the SIMO hardware to be able to have proper timing\n"
 		(exclude_from_sim no)
-		(at 200.66 99.695 0)
-		(size 24.13 17.145)
+		(at 198.755 106.68 0)
+		(size 33.02 12.7)
 		(stroke
 			(width 0)
@@
 	(text_box "P1.6 is used as an alternate timer TA01 pin for the RC PWM output"
 		(exclude_from_sim no)
-		(at 200.66 86.995 0)
-		(size 23.495 11.43)
+		(at 198.755 97.155 0)
+		(size 33.02 7.62)
 		(stroke
 			(width 0)
@@
 		(on_board yes)
 		(dnp no)
-		(fields_autoplaced yes)
 		(property "Reference" "H1"
-			(at 29.21 146.0499 0)
+			(at 29.21 146.05 0)
 			(effects
 				(font

Commit message: later
Connections:
- net +3V3: no longer J3.1 (Pin_1)
- net GND: now also J3.1 (Pin_1)
Changed lines of the file:
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@@
 	(wire
 		(pts
+			(xy 210.82 30.48) (xy 210.82 31.75)
+		)
+		(stroke
+			(width 0)
+			(type default)
+		)
+	)
+	(wire
+		(pts
 			(xy 58.42 44.45) (xy 68.58 44.45)
 		)
@@
 	(wire
 		(pts
+			(xy 215.9 35.56) (xy 215.9 30.48)
+		)
+		(stroke
+			(width 0)
+			(type default)
+		)
+	)
+	(wire
+		(pts
 			(xy 36.83 96.52) (xy 36.83 106.68)
 		)
@@
 	(wire
 		(pts
-			(xy 191.77 35.56) (xy 191.77 33.02)
-		)
-		(stroke
-			(width 0)
-			(type default)
-		)
-	)
-	(wire
-		(pts
 			(xy 68.58 35.56) (xy 68.58 36.83)
 		)
@@
 	(wire
 		(pts
-			(xy 261.62 78.74) (xy 261.62 81.28)
+			(xy 215.9 30.48) (xy 210.82 30.48)
 		)
 		(stroke
@@
 	(wire
 		(pts
-			(xy 53.34 93.98) (xy 55.88 93.98)
+			(xy 261.62 78.74) (xy 261.62 81.28)
 		)
 		(stroke
@@
 	(wire
 		(pts
-			(xy 55.88 93.98) (xy 55.88 91.44)
+			(xy 53.34 93.98) (xy 55.88 93.98)
 		)
 		(stroke
@@
 	(wire
 		(pts
-			(xy 259.08 83.82) (xy 261.62 83.82)
+			(xy 55.88 93.98) (xy 55.88 91.44)
 		)
 		(stroke
@@
 	(wire
 		(pts
-			(xy 243.84 78.74) (xy 243.84 81.28)
+			(xy 259.08 83.82) (xy 261.62 83.82)
 		)
 		(stroke
@@
 	(wire
 		(pts
-			(xy 38.1 81.28) (xy 40.64 81.28)
+			(xy 243.84 78.74) (xy 243.84 81.28)
 		)
 		(stroke
@@
 	(wire
 		(pts
-			(xy 273.05 99.06) (xy 273.05 120.65)
+			(xy 38.1 81.28) (xy 40.64 81.28)
 		)
 		(stroke
@@
 	(wire
 		(pts
-			(xy 105.41 44.45) (xy 105.41 41.91)
+			(xy 273.05 99.06) (xy 273.05 120.65)
 		)
 		(stroke
@@
 	(wire
 		(pts
-			(xy 191.77 35.56) (xy 215.9 35.56)
+			(xy 105.41 44.45) (xy 105.41 41.91)
 		)
 		(stroke
@@
 	)
 	(symbol
+		(lib_id "power:GND")
+		(at 210.82 31.75 0)
+		(unit 1)
+		(exclude_from_sim no)
+		(in_bom yes)
+		(on_board yes)
+		(dnp no)
+		(property "Reference" "#PWR017"
+			(at 210.82 38.1 0)
+			(effects
+				(font
+					(size 1.27 1.27)
+				)
+				(hide yes)
+			)
+		)
+		(property "Value" "GND"
+			(at 208.28 31.75 0)
+			(effects
+				(font
+					(size 1.27 1.27)
+				)
+			)
+		)
+		(property "Footprint" ""
+			(at 210.82 31.75 0)
+			(effects
+				(font
+					(size 1.27 1.27)
+				)
+				(hide yes)
+			)
+		)
+		(property "Datasheet" ""
+			(at 210.82 31.75 0)
+			(effects
+				(font
+					(size 1.27 1.27)
+				)
+				(hide yes)
+			)
+		)
+		(property "Description" "Power symbol creates a global label with name \"GND\" , ground"
+			(at 210.82 31.75 0)
+			(effects
+				(font
+					(size 1.27 1.27)
+				)
+				(hide yes)
+			)
+		)
+		(pin "1"
+		)
+		(instances
+			(project "Wooden_Mirror"
+				(path "/4a0118d4-2192-466c-b388-156d8d14982b"
+					(reference "#PWR017")
+					(unit 1)
+				)
+			)
+		)
+	)
+	(symbol
 		(lib_id "Connector_Generic:Conn_01x05")
 		(at 220.98 40.64 0)
@@
 					(unit 1)
 				)
-			)
-		)
-	)
-	(symbol
-		(lib_id "power:+3V3")
-		(at 191.77 33.02 0)
-		(unit 1)
-		(exclude_from_sim no)
-		(in_bom yes)
-		(on_board yes)
-		(dnp no)
-		(property "Reference" "#PWR017"
-			(at 191.77 36.83 0)
-			(effects
-				(font
-					(size 1.27 1.27)
-				)
-				(hide yes)
-			)
-		)
-		(property "Value" "+3V3"
-			(at 191.77 29.21 0)
-			(effects
-				(font
-					(size 1.27 1.27)
-				)
-			)
-		)
-		(property "Footprint" ""
-			(at 191.77 33.02 0)
-			(effects
-				(font
-					(size 1.27 1.27)
-				)
-				(hide yes)
-			)
-		)
-		(property "Datasheet" ""
-			(at 191.77 33.02 0)
-			(effects
-				(font
-					(size 1.27 1.27)
-				)
-				(hide yes)
-			)
-		)
-		(property "Description" "Power symbol creates a global label with name \"+3V3\""
-			(at 191.77 33.02 0)
-			(effects
-				(font
-					(size 1.27 1.27)
-				)
-				(hide yes)
-			)
-		)
-		(pin "1"
-		)
-		(instances
-			(project "Wooden_Mirror"
-				(path "/4a0118d4-2192-466c-b388-156d8d14982b"
-					(reference "#PWR017")
-					(unit 1)
-				)
